File: _autosave-EMS_stimulator.kicad_pcb (KiCad board)
At the start: 4 copper layers, 42.8 x 33.4 mm, 98 parts, among them IC1 MCP73832, IC2 TPS78230, IC3 MIC5501, IC4 MAX5820, IC5 INA180, IC6 TLV3201, IC7 MAX9619, IC8 TS880ILT, J1 USB_B_micro, P1 TAG connector 2x3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

Commit message: Update schematic with switches neccesary to generate two different voltages on separate capacitors.
Parts:
- removed D2: 1A, 600mV, WL_diodes:SOD-123FL
- added Q10: PNP_BEC, WL_transistors_smd:SOT-23-3, B.Cu at (72.1, 97.3)
- added Q11: NMOS, WL_transistors_smd:SOT-346, B.Cu at (67.6, 97.2)
- added Q12: PNP_BEC, WL_transistors_smd:SOT-23-3, B.Cu at (80.8, 125.8)
- added Q13: NMOS, WL_transistors_smd:SOT-346, B.Cu at (80.9, 120.5)
- added R39: 47, WL_passives:R0402, B.Cu at (71.6, 91.7)
- added R40: 330K, WL_passives:R0402, B.Cu at (80.5, 98.3)
- added R41: 33K, WL_passives:R0402, B.Cu at (80.3, 123.3)
- added R42: 33K, WL_passives:R0402, F.Cu at (112.0, 99.8)
- added R43: 47, WL_passives:R0402, B.Cu at (80.9, 116.5)
- added R44: 330K, WL_passives:R0402, B.Cu at (80.9, 117.9)
- R35: value 2k2 -> 33K; moved to B.Cu
- R36: value 2k2 -> 33K
- moved R35 28.8 mm to (71.6, 94.0), turned to 0 degrees
- moved R36 12.2 mm to (99.8, 99.8), turned to 90 degrees
Connections:
- C9 pad 2: Net-(C13-Pad1) -> GND
- IC2 pad : GND -> (no net)
- L1 pad 2: Net-(D2-Pad1) -> Net-(L1-Pad2)
- Q2 pad 3: Net-(D2-Pad1) -> Net-(L1-Pad2)
- R35 pad 1: Net-(Q4-Pad3) -> Net-(Q10-Pad1)
- R35 pad 2: Net-(Q1-Pad1) -> Net-(Q11-Pad3)
- R36 pad 1: Net-(Q7-Pad3) -> Net-(Q1-Pad1)
- R36 pad 2: Net-(Q5-Pad1) -> Net-(Q4-Pad3)
- R8 pad 1: Net-(C9-Pad1) -> Net-(L1-Pad2)
- TP4 pad 1: Net-(D2-Pad1) -> Net-(L1-Pad2)
Routing:
- net Net-(L1-Pad2): track 0.00 -> 15.1 mm, vias 0 -> 1
- net Net-(D2-Pad1): track 11.5 -> 0.00 mm
- net Net-(C9-Pad1): track 15.4 -> 11.8 mm, vias 6 -> 5
